File: _saved_Sumozinho.sch (KiCad schematic (older format))
At the start: 17 parts, among them U1 STM32F103C8T6, U2 lm393, U3 tcrt5000, U4 tcrt5000, U5 l298mini, U6 lm393, U7 lm393, U8 tcrt5000, U9 tcrt5000

Commit message: Adds new footprints
Parts:
- U2, U6, U7: footprint (none) -> lm393:lm393
- U3, U4, U8, U9: footprint (none) -> tcrt5000:tcrt5000
- U5: footprint (none) -> l298nmini:l298nmini
Changed lines of the file:
@@
 F 0 "U4" H 4800 5550 60  0000 C CNN
 F 1 "tcrt5000" H 4700 5650 60  0000 C CNN
-F 2 "" H 4900 5700 60  0001 C CNN
+F 2 "tcrt5000:tcrt5000" H 4900 5700 60  0001 C CNN
 F 3 "" H 4900 5700 60  0001 C CNN
 	1    4900 5700
@@
 F 0 "U7" H 7450 3850 60  0000 C CNN
 F 1 "lm393" H 7450 3750 60  0000 C CNN
-F 2 "" H 7300 3700 60  0001 C CNN
+F 2 "lm393:lm393" H 7300 3700 60  0001 C CNN
 F 3 "" H 7300 3700 60  0001 C CNN
 	1    7300 3700
@@
 F 0 "U2" H 4550 3900 60  0000 C CNN
 F 1 "lm393" H 4550 3800 60  0000 C CNN
-F 2 "" H 4400 3750 60  0001 C CNN
+F 2 "lm393:lm393" H 4400 3750 60  0001 C CNN
 F 3 "" H 4400 3750 60  0001 C CNN
 	1    4400 3750
@@
 F 0 "U6" V 6450 5850 60  0000 C CNN
 F 1 "lm393" H 6450 5750 60  0000 C CNN
-F 2 "" H 6300 5700 60  0001 C CNN
+F 2 "lm393:lm393" H 6300 5700 60  0001 C CNN
 F 3 "" H 6300 5700 60  0001 C CNN
 	1    6300 5700
@@
 F 0 "U9" H 7300 5500 60  0000 C CNN
 F 1 "tcrt5000" H 7200 5600 60  0000 C CNN
-F 2 "" H 7400 5650 60  0001 C CNN
+F 2 "tcrt5000:tcrt5000" H 7400 5650 60  0001 C CNN
 F 3 "" H 7400 5650 60  0001 C CNN
 	1    7400 5650
@@
 F 0 "U3" H 4400 2000 60  0000 C CNN
 F 1 "tcrt5000" H 4300 2100 60  0000 C CNN
-F 2 "" H 4500 2150 60  0001 C CNN
+F 2 "tcrt5000:tcrt5000" H 4500 2150 60  0001 C CNN
 F 3 "" H 4500 2150 60  0001 C CNN
 	1    4500 2150
@@
 F 0 "U8" H 7250 2000 60  0000 C CNN
 F 1 "tcrt5000" H 7150 2100 60  0000 C CNN
-F 2 "" H 7350 2150 60  0001 C CNN
+F 2 "tcrt5000:tcrt5000" H 7350 2150 60  0001 C CNN
 F 3 "" H 7350 2150 60  0001 C CNN
 	1    7350 2150
@@
 F 0 "U5" H 5250 5550 60  0000 C CNN
 F 1 "l298mini" H 5550 5600 60  0000 C CNN
-F 2 "" H 5350 5350 60  0001 C CNN
+F 2 "l298nmini:l298nmini" H 5350 5350 60  0001 C CNN
 F 3 "" H 5350 5350 60  0001 C CNN
 	1    5550 5400
