File: Sumozinho.kicad_pcb (KiCad board)
At the start: 2 copper layers, 0 parts

Commit message: Ratnest ready
Parts:
- added R1: R, Resistors_SMD:R_0805_HandSoldering, F.Cu at (161.3, 35.6)
- added R2: R, Resistors_SMD:R_0805_HandSoldering, F.Cu at (198.1, 64.8)
- added R3: R, Resistors_SMD:R_0805_HandSoldering, F.Cu at (170.2, 27.9)
- added R4: R, Resistors_SMD:R_0805_HandSoldering, F.Cu at (138.4, 39.4)
- added R5: R, Resistors_SMD:R_0805_HandSoldering, F.Cu at (191.8, 83.8)
- added R6: R, Resistors_SMD:R_0805_HandSoldering, F.Cu at (177.8, 26.7)
- added R7: R, Resistors_SMD:R_0805_HandSoldering, F.Cu at (154.9, 35.6)
- added R8: R, Resistors_SMD:R_0805_HandSoldering, F.Cu at (163.8, 83.8)
- added U1: STM32F103C8T6, stm32:stm32, F.Cu at (175.3, 53.3)
- added U2: lm393, lm393:lm393, F.Cu at (181.6, 67.3)
- added U3: tcrt5000, tcrt5000:tcrt5000, F.Cu at (115.6, 36.8)
- added U4: tcrt5000, tcrt5000:tcrt5000, F.Cu at (115.6, 81.3)
- added U5: l298mini, l298nmini:l298nmini, F.Cu at (182.9, 141.0)
- added U6: lm393, lm393:lm393, F.Cu at (147.3, 96.5)
- added U7: lm393, lm393:lm393, F.Cu at (96.5, 72.4)
- added U8: tcrt5000, tcrt5000:tcrt5000, F.Cu at (171.4, 38.1)
- added U9: tcrt5000, tcrt5000:tcrt5000, F.Cu at (147.3, 123.2)
