File: Sumozinho.kicad_pcb (KiCad board)
At the start: 2 copper layers, 17 parts, among them U1 STM32F103C8T6, U2 lm393, U3 tcrt5000, U4 tcrt5000, U5 l298mini, U6 lm393, U7 lm393, U8 tcrt5000, U9 tcrt5000

Commit message: Auto stash before merge of "master" and "origin/master"
Parts:
- moved U5 43.7 mm to (157.5, 91.4)
- moved U9 43.3 mm to (175.3, 90.2)
- moved U4 19.0 mm to (115.6, 100.3)
Changed lines of the file:
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@@
     (links 39)
     (no_connects 39)
-    (area 0 0 0 0)
+    (area 95.045 24.094999 200.695001 131.562021)
     (thickness 1.6)
     (drawings 0)
@@
   )
   (module l298nmini:l298nmini (layer F.Cu)
-    (at 193.04 116.84 270)
+    (at 157.48 91.44 270)
     (fp_text reference U5 (at 0 0.5 270) (layer F.SilkS)
       (effects (font (size 1 1) (thickness 0.15)))
@@
   )
   (module tcrt5000:tcrt5000 (layer F.Cu)
-    (at 115.57 81.28)
+    (at 115.57 100.33)
     (fp_text reference U4 (at 0 0.5) (layer F.SilkS)
       (effects (font (size 1 1) (thickness 0.15)))
@@
   )
   (module tcrt5000:tcrt5000 (layer F.Cu)
-    (at 147.32 123.19)
+    (at 175.26 90.17)
     (fp_text reference U9 (at 0 0.5) (layer F.SilkS)
       (effects (font (size 1 1) (thickness 0.15)))

Commit message: Hot fixes
Parts:
- R1, R2, R3, R4, R5, R6, R7, R8: footprint Resistors_SMD:R_0805_HandSoldering -> resistor:R_0805_HandSoldering
- U5: footprint l298nmini:l298nmini -> l298mini:l298nmini
- moved R2 81.6 mm to (131.1, 111.3), turned to 180 degrees
- moved R4 73.0 mm to (125.5, 111.3)
- moved R3 65.9 mm to (104.6, 34.8)
- moved R1 50.3 mm to (111.0, 34.8)
- moved U5 46.5 mm to (154.3, 45.1), turned to 0 degrees
- moved R5 41.1 mm to (160.8, 110.7)
- moved U9 34.5 mm to (163.8, 122.7), turned to 180 degrees
- moved R7 33.0 mm to (188.0, 36.8), turned to 180 degrees
- moved U7 29.9 mm to (123.4, 59.4), turned to 0 degrees
- moved R8 27.0 mm to (166.1, 110.7), turned to 180 degrees
- moved U4 26.1 mm to (129.0, 122.7), turned to 180 degrees
- moved U8 16.9 mm to (185.4, 47.6), turned to 180 degrees
- moved U2 15.5 mm to (169.9, 77.5), turned to 180 degrees
- moved U3 11.9 mm to (108.2, 46.2), turned to 180 degrees
- moved R6 10.9 mm to (181.6, 36.8), turned to 180 degrees
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Connections:
- R6 pad 1: VCC -> (no net)
Routing:
- net Net-(R1-Pad1): track 0.00 -> 142.5 mm
- net Net-(R2-Pad1): track 0.00 -> 138.8 mm
- net Net-(R8-Pad1): track 0.00 -> 99.5 mm
- net Net-(R7-Pad1): track 0.00 -> 84.6 mm
- net Net-(U1-Pad31): track 0.00 -> 71.6 mm
- net Net-(U1-Pad40): track 0.00 -> 15.7 mm
- net Net-(U1-Pad24): track 0.00 -> 14.3 mm
- net Net-(U1-Pad36): track 0.00 -> 14.3 mm
- net Net-(U1-Pad37): track 0.00 -> 14.2 mm
- net Net-(U1-Pad32): track 0.00 -> 12.3 mm
- net Net-(U1-Pad33): track 0.00 -> 12.2 mm
- net Net-(R5-Pad1): track 0.00 -> 10.9 mm
- net Net-(R4-Pad1): track 0.00 -> 10.8 mm
- net Net-(R3-Pad2): track 0.00 -> 10.2 mm
- net Net-(R6-Pad2): track 0.00 -> 9.24 mm
- added copper zone on B.Cu, net GND
- added copper zone on F.Cu, net VCC
Other:
- net class Default: clearance 0.2 -> 0.6; trace_width 0.25 -> 0.8
- rule trace_clearance: 0.2 -> 0.6
