File: _autosave-Sumozinho.kicad_pcb (KiCad board)
At the start: 2 copper layers, 17 parts, among them U1 STM32F103C8T6, U2 lm393, U3 tcrt5000, U4 tcrt5000, U5 l298mini, U6 lm393, U7 lm393, U8 tcrt5000, U9 tcrt5000

Commit message: Minor changes
Parts:
- moved U5 59.7 mm to (146.1, 80.0), turned to 0 degrees
Changed lines of the file:
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@@
     (links 39)
     (no_connects 39)
-    (area 0 0 0 0)
+    (area 95.045 24.094999 200.695001 131.562021)
     (thickness 1.6)
     (drawings 0)
@@
   )
   (module l298nmini:l298nmini (layer F.Cu)
-    (at 193.04 116.84 270)
-    (fp_text reference U5 (at 0 0.5 270) (layer F.SilkS)
-      (effects (font (size 1 1) (thickness 0.15)))
-    )
-    (fp_text value l298mini (at 0 -0.5 270) (layer F.Fab)
+    (at 146.05 80.01)
+    (fp_text reference U5 (at 0 0.5) (layer F.SilkS)
+      (effects (font (size 1 1) (thickness 0.15)))
+    )
+    (fp_text value l298mini (at 0 -0.5) (layer F.Fab)
       (effects (font (size 1 1) (thickness 0.15)))
     )
@@
     (fp_line (start -8.35406 5.66674) (end 8.85698 5.61086) (layer F.SilkS) (width 0.15))
     (fp_line (start 8.85698 5.61086) (end 8.82904 1.67132) (layer F.SilkS) (width 0.15))
-    (pad 1 smd circle (at -4.191 3.1242 270) (size 1.524 1.524) (layers F.Cu F.Paste F.Mask)
+    (pad 1 smd circle (at -4.191 3.1242) (size 1.524 1.524) (layers F.Cu F.Paste F.Mask)
       (net 12 "Net-(U1-Pad32)"))
-    (pad 2 smd circle (at -1.397 3.1242 270) (size 1.524 1.524) (layers F.Cu F.Paste F.Mask)
+    (pad 2 smd circle (at -1.397 3.1242) (size 1.524 1.524) (layers F.Cu F.Paste F.Mask)
       (net 13 "Net-(U1-Pad33)"))
-    (pad 3 smd circle (at 1.31318 3.06832 270) (size 1.524 1.524) (layers F.Cu F.Paste F.Mask)
+    (pad 3 smd circle (at 1.31318 3.06832) (size 1.524 1.524) (layers F.Cu F.Paste F.Mask)
       (net 14 "Net-(U1-Pad36)"))
-    (pad 4 smd circle (at 3.9116 3.09626 270) (size 1.524 1.524) (layers F.Cu F.Paste F.Mask)
+    (pad 4 smd circle (at 3.9116 3.09626) (size 1.524 1.524) (layers F.Cu F.Paste F.Mask)
       (net 15 "Net-(U1-Pad37)"))
   )
