File: Sumozinho.sch (KiCad schematic (older format))
At the start: 17 parts, among them U1 STM32F103C8T6, U2 lm393, U3 tcrt5000, U4 tcrt5000, U5 l298mini, U6 lm393, U7 lm393, U8 tcrt5000, U9 tcrt5000

Commit message: Ratnest ready
Parts:
- U1: footprint stm32f103c8t6:stm32 -> stm32:stm32
- U2, U6, U7: footprint (none) -> lm393:lm393
- U3, U4, U8, U9: footprint (none) -> tcrt5000:tcrt5000
- U5: footprint (none) -> l298nmini:l298nmini
Connections:
- wire segments 44 -> 47
Changed lines of the file:
@@
 F 0 "U1" H 6150 5000 60  0000 C CNN
 F 1 "STM32F103C8T6" H 6150 2800 60  0000 C CNN
-F 2 "stm32f103c8t6:stm32" H 6150 5050 60  0001 C CNN
+F 2 "stm32:stm32" H 6150 5050 60  0001 C CNN
 F 3 "" H 6150 5050 60  0001 C CNN
 	1    6150 3950
@@
 F 0 "U4" H 4800 5550 60  0000 C CNN
 F 1 "tcrt5000" H 4700 5650 60  0000 C CNN
-F 2 "" H 4900 5700 60  0001 C CNN
+F 2 "tcrt5000:tcrt5000" H 4900 5700 60  0001 C CNN
 F 3 "" H 4900 5700 60  0001 C CNN
 	1    4900 5700
@@
 F 0 "U7" H 7450 3850 60  0000 C CNN
 F 1 "lm393" H 7450 3750 60  0000 C CNN
-F 2 "" H 7300 3700 60  0001 C CNN
+F 2 "lm393:lm393" H 7300 3700 60  0001 C CNN
 F 3 "" H 7300 3700 60  0001 C CNN
 	1    7300 3700
@@
 F 0 "U2" H 4550 3900 60  0000 C CNN
 F 1 "lm393" H 4550 3800 60  0000 C CNN
-F 2 "" H 4400 3750 60  0001 C CNN
+F 2 "lm393:lm393" H 4400 3750 60  0001 C CNN
 F 3 "" H 4400 3750 60  0001 C CNN
 	1    4400 3750
@@
 F 0 "U6" V 6450 5850 60  0000 C CNN
 F 1 "lm393" H 6450 5750 60  0000 C CNN
-F 2 "" H 6300 5700 60  0001 C CNN
+F 2 "lm393:lm393" H 6300 5700 60  0001 C CNN
 F 3 "" H 6300 5700 60  0001 C CNN
 	1    6300 5700
@@
 F 0 "U9" H 7300 5500 60  0000 C CNN
 F 1 "tcrt5000" H 7200 5600 60  0000 C CNN
-F 2 "" H 7400 5650 60  0001 C CNN
+F 2 "tcrt5000:tcrt5000" H 7400 5650 60  0001 C CNN
 F 3 "" H 7400 5650 60  0001 C CNN
 	1    7400 5650
@@
 F 0 "U3" H 4400 2000 60  0000 C CNN
 F 1 "tcrt5000" H 4300 2100 60  0000 C CNN
-F 2 "" H 4500 2150 60  0001 C CNN
+F 2 "tcrt5000:tcrt5000" H 4500 2150 60  0001 C CNN
 F 3 "" H 4500 2150 60  0001 C CNN
 	1    4500 2150
@@
 F 0 "U8" H 7250 2000 60  0000 C CNN
 F 1 "tcrt5000" H 7150 2100 60  0000 C CNN
-F 2 "" H 7350 2150 60  0001 C CNN
+F 2 "tcrt5000:tcrt5000" H 7350 2150 60  0001 C CNN
 F 3 "" H 7350 2150 60  0001 C CNN
 	1    7350 2150
@@
 F 0 "U5" H 5250 5550 60  0000 C CNN
 F 1 "l298mini" H 5550 5600 60  0000 C CNN
-F 2 "" H 5350 5350 60  0001 C CNN
+F 2 "l298nmini:l298nmini" H 5350 5350 60  0001 C CNN
 F 3 "" H 5350 5350 60  0001 C CNN
 	1    5550 5400
@@
 Wire Wire Line
 	7900 3400 7900 3450
+Wire Wire Line
+	7900 5300 7900 5350
+Wire Wire Line
+	4150 5400 4150 5450
+Wire Wire Line
+	7400 1600 7400 1650
 $EndSCHEMATC

Commit message: Auto stash before merge of "master" and "origin/master"
Parts:
- U3, U4, U8, U9: footprint tcrt5000:tcrt5000 -> lm393:tcrt5000
Connections:
- wire segments 47 -> 46
Changed lines of the file:
@@
 F 0 "U4" H 4800 5550 60  0000 C CNN
 F 1 "tcrt5000" H 4700 5650 60  0000 C CNN
-F 2 "tcrt5000:tcrt5000" H 4900 5700 60  0001 C CNN
+F 2 "lm393:tcrt5000" H 4900 5700 60  0001 C CNN
 F 3 "" H 4900 5700 60  0001 C CNN
 	1    4900 5700
@@
 F 0 "U9" H 7300 5500 60  0000 C CNN
 F 1 "tcrt5000" H 7200 5600 60  0000 C CNN
-F 2 "tcrt5000:tcrt5000" H 7400 5650 60  0001 C CNN
+F 2 "lm393:tcrt5000" H 7400 5650 60  0001 C CNN
 F 3 "" H 7400 5650 60  0001 C CNN
 	1    7400 5650
@@
 F 0 "U3" H 4400 2000 60  0000 C CNN
 F 1 "tcrt5000" H 4300 2100 60  0000 C CNN
-F 2 "tcrt5000:tcrt5000" H 4500 2150 60  0001 C CNN
+F 2 "lm393:tcrt5000" H 4500 2150 60  0001 C CNN
 F 3 "" H 4500 2150 60  0001 C CNN
 	1    4500 2150
@@
 F 0 "U8" H 7250 2000 60  0000 C CNN
 F 1 "tcrt5000" H 7150 2100 60  0000 C CNN
-F 2 "tcrt5000:tcrt5000" H 7350 2150 60  0001 C CNN
+F 2 "lm393:tcrt5000" H 7350 2150 60  0001 C CNN
 F 3 "" H 7350 2150 60  0001 C CNN
 	1    7350 2150
@@
 	7900 3400 7900 3450
 Wire Wire Line
+	4150 5400 4150 5450
+Wire Wire Line
 	7900 5300 7900 5350
-Wire Wire Line
-	4150 5400 4150 5450
-Wire Wire Line
-	7400 1600 7400 1650
 $EndSCHEMATC

Commit message: Hot fixes
Parts:
- R1, R2, R3, R4, R5, R6, R7, R8: footprint Resistors_SMD:R_0805_HandSoldering -> resistor:R_0805_HandSoldering
- U3, U4, U8, U9: footprint lm393:tcrt5000 -> tcrt5000:tcrt5000
- U5: footprint l298nmini:l298nmini -> l298mini:l298nmini
Changed lines of the file:
@@
 F 0 "U4" H 4800 5550 60  0000 C CNN
 F 1 "tcrt5000" H 4700 5650 60  0000 C CNN
-F 2 "lm393:tcrt5000" H 4900 5700 60  0001 C CNN
+F 2 "tcrt5000:tcrt5000" H 4900 5700 60  0001 C CNN
 F 3 "" H 4900 5700 60  0001 C CNN
 	1    4900 5700
@@
 F 0 "U9" H 7300 5500 60  0000 C CNN
 F 1 "tcrt5000" H 7200 5600 60  0000 C CNN
-F 2 "lm393:tcrt5000" H 7400 5650 60  0001 C CNN
+F 2 "tcrt5000:tcrt5000" H 7400 5650 60  0001 C CNN
 F 3 "" H 7400 5650 60  0001 C CNN
 	1    7400 5650
@@
 F 0 "U3" H 4400 2000 60  0000 C CNN
 F 1 "tcrt5000" H 4300 2100 60  0000 C CNN
-F 2 "lm393:tcrt5000" H 4500 2150 60  0001 C CNN
+F 2 "tcrt5000:tcrt5000" H 4500 2150 60  0001 C CNN
 F 3 "" H 4500 2150 60  0001 C CNN
 	1    4500 2150
@@
 F 0 "U8" H 7250 2000 60  0000 C CNN
 F 1 "tcrt5000" H 7150 2100 60  0000 C CNN
-F 2 "lm393:tcrt5000" H 7350 2150 60  0001 C CNN
+F 2 "tcrt5000:tcrt5000" H 7350 2150 60  0001 C CNN
 F 3 "" H 7350 2150 60  0001 C CNN
 	1    7350 2150
@@
 F 0 "R2" V 4230 5250 50  0000 C CNN
 F 1 "R" V 4150 5250 50  0000 C CNN
-F 2 "Resistors_SMD:R_0805_HandSoldering" V 4080 5250 50  0001 C CNN
+F 2 "resistor:R_0805_HandSoldering" V 4080 5250 50  0001 C CNN
 F 3 "" H 4150 5250 50  0001 C CNN
 	1    4150 5250
@@
 F 0 "R8" V 7980 5150 50  0000 C CNN
 F 1 "R" V 7900 5150 50  0000 C CNN
-F 2 "Resistors_SMD:R_0805_HandSoldering" V 7830 5150 50  0001 C CNN
+F 2 "resistor:R_0805_HandSoldering" V 7830 5150 50  0001 C CNN
 F 3 "" H 7900 5150 50  0001 C CNN
 	1    7900 5150
@@
 F 0 "R1" V 4230 3150 50  0000 C CNN
 F 1 "R" V 4150 3150 50  0000 C CNN
-F 2 "Resistors_SMD:R_0805_HandSoldering" V 4080 3150 50  0001 C CNN
+F 2 "resistor:R_0805_HandSoldering" V 4080 3150 50  0001 C CNN
 F 3 "" H 4150 3150 50  0001 C CNN
 	1    4150 3150
@@
 F 0 "R7" V 7980 3250 50  0000 C CNN
 F 1 "R" V 7900 3250 50  0000 C CNN
-F 2 "Resistors_SMD:R_0805_HandSoldering" V 7830 3250 50  0001 C CNN
+F 2 "resistor:R_0805_HandSoldering" V 7830 3250 50  0001 C CNN
 F 3 "" H 7900 3250 50  0001 C CNN
 	1    7900 3250
@@
 F 0 "R6" V 7480 1800 50  0000 C CNN
 F 1 "R" V 7400 1800 50  0000 C CNN
-F 2 "Resistors_SMD:R_0805_HandSoldering" V 7330 1800 50  0001 C CNN
+F 2 "resistor:R_0805_HandSoldering" V 7330 1800 50  0001 C CNN
 F 3 "" H 7400 1800 50  0001 C CNN
 	1    7400 1800
@@
 F 0 "R3" V 4630 1800 50  0000 C CNN
 F 1 "R" V 4550 1800 50  0000 C CNN
-F 2 "Resistors_SMD:R_0805_HandSoldering" V 4480 1800 50  0001 C CNN
+F 2 "resistor:R_0805_HandSoldering" V 4480 1800 50  0001 C CNN
 F 3 "" H 4550 1800 50  0001 C CNN
 	1    4550 1800
@@
 F 0 "R4" V 4930 6050 50  0000 C CNN
 F 1 "R" V 4850 6050 50  0000 C CNN
-F 2 "Resistors_SMD:R_0805_HandSoldering" V 4780 6050 50  0001 C CNN
+F 2 "resistor:R_0805_HandSoldering" V 4780 6050 50  0001 C CNN
 F 3 "" H 4850 6050 50  0001 C CNN
 	1    4850 6050
@@
 F 0 "R5" V 7430 6050 50  0000 C CNN
 F 1 "R" V 7350 6050 50  0000 C CNN
-F 2 "Resistors_SMD:R_0805_HandSoldering" V 7280 6050 50  0001 C CNN
+F 2 "resistor:R_0805_HandSoldering" V 7280 6050 50  0001 C CNN
 F 3 "" H 7350 6050 50  0001 C CNN
 	1    7350 6050
@@
 F 0 "U5" H 5250 5550 60  0000 C CNN
 F 1 "l298mini" H 5550 5600 60  0000 C CNN
-F 2 "l298nmini:l298nmini" H 5350 5350 60  0001 C CNN
+F 2 "l298mini:l298nmini" H 5350 5350 60  0001 C CNN
 F 3 "" H 5350 5350 60  0001 C CNN
 	1    5550 5400
